Commit message: created robot

File: description/lidar.xacro (robot description, xacro)
@@ -26,5 +26,5 @@
         <sensor name="laser" type="ray">
             <pose> 0 0 0 0 0 0 </pose>
-            <visualize>false</visualize>
+            <visualize>true</visualize>
             <update_rate>10</update_rate>
             <ray>

File: description/robot_core.xacro (robot description, xacro)
@@ -19,4 +19,12 @@
     <!-- BASE LINK -->
     <link name="base_link">
+    </link>
+   <!-- BASE_FOOTPRINT LINK -->
+    <joint name="base_footprint_joint" type="fixed">
+        <parent link="base_link"/>
+        <child link="base_footprint"/>
+        <origin xyz="0 0 0" rpy="0 0 0"/>
+    </joint>
+    <link name="base_footprint">
     </link>
     <!-- CHASSIS LINK -->
@@ -196,4 +204,5 @@
 ros2 run teleop_twist_keyboard teleop_twist_keyboard
 ros2 topic echo /cmd_vel
+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
 ros2 run rplidar_ros rplidar_composition -ros-args -p serial_port:=/dev/serial/by-path/platform-fd500000.pcie-pci-0000:01:00.0-usb-0:1.3:1.0-port0 -p frame_id:=laser_frame -p angle_compensate:=true -p scan_mode:=Standard
 -->
@@ -202,2 +211,8 @@
 we have in our hand a tool that can convert URDF to sdf in order to get the entity
 spawned in the gazebo environnement -->
+                        <!-- SLAM -->
+<!-- we use the grid slam not the one with features and what we do is we pixalize the world and each one of the places whe associate a probabilities of occupation
+AMCL : adaptive monto carlo localisation (we need a map in order to do the localisation )
+ros2 run nav2_util lifecycle_bringup map_server
+ros2 run nav2_amcl amcl -ros-args -p use_sim_time:=true
+ros2 run nav2_map_server map_server -ros-args -p yaml_filename:=my_map_save.yaml -p use_sim_time:=true  (is for the creation of the node that will broadcast the /map topic) -->
