Commit message: last modify

File: description/camera.xacro (robot description, xacro)
@@ -4,5 +4,5 @@
         <parent link="chassis"/>
         <child link="camera_link"/>
-        <origin xyz="0.405 0 0.08" rpy="0 0 0"/>
+        <origin xyz="0.265 0 0.08" rpy="0 0 0"/>
     </joint>
     <link name="camera_link">

File: description/lidar.xacro (robot description, xacro)
@@ -4,10 +4,10 @@
         <parent link="chassis"/>
         <child link="laser_frame"/>
-        <origin xyz="0.2 0 0.175" rpy="0 0 0"/>
+        <origin xyz="0.13 0 0.065" rpy="0 0 0"/>
     </joint>
     <link name="laser_frame">
         <visual>
             <geometry>
-                <cylinder radius="0.05" length="0.04"/>
+                <cylinder radius="0.03" length="0.026"/>
             </geometry>
             <material name="red"/>
@@ -15,8 +15,8 @@
         <collision>
             <geometry>
-                <cylinder radius="0.05" length="0.04"/>
+                <cylinder radius="0.03" length="0.026"/>
             </geometry>
         </collision>
-        <xacro:inertial_cylinder mass="0.1" length="0.04" radius="0.05">
+        <xacro:inertial_cylinder mass="0.05" length="0.026" radius="0.03">
             <origin xyz="0 0 0" rpy="0 0 0"/>
         </xacro:inertial_cylinder>

File: description/robot.urdf.xacro (robot description, xacro)
@@ -1,6 +1,12 @@
 <?xml version="1.0"?>
 <robot xmlns:xacro="http://www.ros.org/wiki/xacro"  name="robot">
+    <xacro:arg name="use_ros2_control" default="true"/>
     <xacro:include filename="robot_core.xacro" />
-    <xacro:include filename="gazebo_control.xacro" />
+    <xacro:if value="$(arg use_ros2_control)">
+        <xacro:include filename="ros2_control.xacro" />
+    </xacro:if>
+    <xacro:unless value="$(arg use_ros2_control)">
+        <xacro:include filename="gazebo_control.xacro" />
+    </xacro:unless>
     <xacro:include filename="lidar.xacro" />
     <xacro:include filename="camera.xacro" />

File: description/robot_core.xacro (robot description, xacro)
@@ -29,25 +29,25 @@
     </link>
     <!-- CHASSIS LINK -->
-    <joint name="chassis_joint" type="fixed">
+     <joint name="chassis_joint" type="fixed">
         <parent link="base_link"/>
         <child link="chassis"/>
-        <origin xyz="-0.1 0 0"/>
+        <origin xyz="-0.075 0 0"/>
     </joint>
     <link name="chassis">
         <visual>
-            <origin xyz="0.2 0 0.075"/>
-            <geometry>
-                <box size="0.4 0.3 0.15"/>
+            <origin xyz="0.13 0 0.0325"/>
+            <geometry>
+                <box size="0.26 0.15 0.065"/>
             </geometry>
             <material name="black"/>
         </visual>
         <collision>
-            <origin xyz="0.2 0 0.075"/>
-            <geometry>
-                <box size="0.4 0.3 0.15"/>
-            </geometry>
-        </collision>
-        <xacro:inertial_box mass="0.5" x="0.4" y="0.3" z="0.15">
-            <origin xyz="0.2 0 0.075" rpy="0 0 0"/>
+            <origin xyz="0.13 0 0.0325"/>
+            <geometry>
+                <box size="0.26 0.15 0.065"/>
+            </geometry>
+        </collision>
+        <xacro:inertial_box mass="0.5" x="0.26" y="0.1" z="0.065">
+            <origin xyz="0.13 0 0.0325" rpy="0 0 0"/>
         </xacro:inertial_box>
     </link>
@@ -60,5 +60,5 @@
         <parent link="base_link"/>
         <child link="left_wheel_back"/>
-        <origin xyz="0 0.175 0" rpy="-${pi/2} 0 0" />
+        <origin xyz="0 0.090 0" rpy="-${pi/2} 0 0" />
         <axis xyz="0 0 1"/>
     </joint>
@@ -66,14 +66,14 @@
         <visual>
             <geometry>
-                <cylinder radius="0.05" length="0.04"/>
-            </geometry>
-            <material name="blue"/>
-        </visual>
-        <collision>
-            <geometry>
-                <cylinder radius="0.05" length="0.04"/>
-            </geometry>
-        </collision>
-        <xacro:inertial_cylinder mass="0.1" length="0.04" radius="0.05">
+                <cylinder radius="0.03" length="0.026"/>
+            </geometry>
+            <material name="blue"/>
+        </visual>
+        <collision>
+            <geometry>
+                <sphere radius="0.03" />
+            </geometry>
+        </collision>
+        <xacro:inertial_cylinder mass="0.1" length="0.026" radius="0.03">
             <origin xyz="0 0 0" rpy="0 0 0"/>
         </xacro:inertial_cylinder>
@@ -86,19 +86,19 @@
         <parent link="base_link"/>
         <child link="left_wheel_front"/>
-        <origin xyz="0.2 0.175 0" rpy="-${pi/2} 0 0" />
+        <origin xyz="0.115 0.090 0" rpy="-${pi/2} 0 0" />
     </joint>
     <link name="left_wheel_front">
         <visual>
             <geometry>
-                <cylinder radius="0.05" length="0.04"/>
-            </geometry>
-            <material name="blue"/>
-        </visual>
-        <collision>
-            <geometry>
-                <cylinder radius="0.05" length="0.04"/>
-            </geometry>
-        </collision>
-        <xacro:inertial_cylinder mass="0.1" length="0.04" radius="0.05">
+                <cylinder radius="0.03" length="0.026"/>
+            </geometry>
+            <material name="blue"/>
+        </visual>
+        <collision>
+            <geometry>
+                <sphere radius="0.03" />
+            </geometry>
+        </collision>
+        <xacro:inertial_cylinder mass="0.1" length="0.026" radius="0.03">
             <origin xyz="0 0 0" rpy="0 0 0"/>
         </xacro:inertial_cylinder>
@@ -113,5 +113,5 @@
         <parent link="base_link"/>
         <child link="right_wheel"/>
-        <origin xyz="0 -0.175 0" rpy="${pi/2} 0 0" />
+        <origin xyz="0 -0.090 0" rpy="${pi/2} 0 0" />
         <axis xyz="0 0 -1"/>
     </joint>
@@ -119,14 +119,14 @@
         <visual>
             <geometry>
-                <cylinder radius="0.05" length="0.04"/>
-            </geometry>
-            <material name="blue"/>
-        </visual>
-        <collision>
-            <geometry>
-                <cylinder radius="0.05" length="0.04"/>
-            </geometry>
-        </collision>
-        <xacro:inertial_cylinder mass="0.1" length="0.04" radius="0.05">
+                <cylinder radius="0.03" length="0.026"/>
+            </geometry>
+            <material name="blue"/>
+        </visual>
+        <collision>
+            <geometry>
+                <sphere radius="0.03" />
+            </geometry>
+        </collision>
+        <xacro:inertial_cylinder mass="0.1" length="0.026" radius="0.03">
             <origin xyz="0 0 0" rpy="0 0 0"/>
         </xacro:inertial_cylinder>
@@ -139,19 +139,19 @@
         <parent link="base_link"/>
         <child link="right_wheel_front"/>
-        <origin xyz="0.2 -0.175 0" rpy="${pi/2} 0 0" />
+        <origin xyz="0.1 -0.090 0" rpy="${pi/2} 0 0" />
     </joint>
     <link name="right_wheel_front">
         <visual>
             <geometry>
-                <cylinder radius="0.05" length="0.04"/>
-            </geometry>
-            <material name="blue"/>
-        </visual>
-        <collision>
-            <geometry>
-                <cylinder radius="0.05" length="0.04"/>
-            </geometry>
-        </collision>
-        <xacro:inertial_cylinder mass="0.1" length="0.04" radius="0.05">
+                <cylinder radius="0.03" length="0.026"/>
+            </geometry>
+            <material name="blue"/>
+        </visual>
+        <collision>
+            <geometry>
+                <sphere radius="0.03" />
+            </geometry>
+        </collision>
+        <xacro:inertial_cylinder mass="0.1" length="0.026" radius="0.03">
             <origin xyz="0 0 0" rpy="0 0 0"/>
         </xacro:inertial_cylinder>
