Commit message: working robot

File: description/gazebo_control.xacro (robot description, xacro)
@@ -6,8 +6,8 @@
             <left_joint>left_wheel_joint</left_joint>
             <right_joint>right_wheel_joint</right_joint>
-            <wheel_separation>0.35</wheel_separation>
-            <wheel_diameter>0.1</wheel_diameter>
+            <wheel_separation>0.18</wheel_separation>
+            <wheel_diameter>0.0325</wheel_diameter>
             <!-- Limits -->
-            <max_wheel_torque>200</max_wheel_torque>
+            <max_wheel_torque>100.0</max_wheel_torque>
             <max_wheel_acceleration>10.0</max_wheel_acceleration>
             <!-- Output -->

File: description/lidar.xacro (robot description, xacro)
@@ -18,5 +18,5 @@
             </geometry>
         </collision>
-        <xacro:inertial_cylinder mass="0.05" length="0.026" radius="0.03">
+        <xacro:inertial_cylinder mass="0.5" length="0.026" radius="0.03">
             <origin xyz="0 0 0" rpy="0 0 0"/>
         </xacro:inertial_cylinder>

File: description/robot.urdf.xacro (robot description, xacro)
@@ -1,4 +1,5 @@
 <?xml version="1.0"?>
 <robot xmlns:xacro="http://www.ros.org/wiki/xacro"  name="robot">
+    <xacro:arg name="sim_mode" default="false"/>
     <xacro:arg name="use_ros2_control" default="true"/>
     <xacro:include filename="robot_core.xacro" />

File: description/robot_core.xacro (robot description, xacro)
@@ -36,18 +36,18 @@
     <link name="chassis">
         <visual>
-            <origin xyz="0.13 0 0.0325"/>
-            <geometry>
-                <box size="0.26 0.15 0.065"/>
+            <origin xyz="0.13 0 0.04"/>
+            <geometry>
+                <box size="0.26 0.15 0.08"/>
             </geometry>
             <material name="black"/>
         </visual>
         <collision>
-            <origin xyz="0.13 0 0.0325"/>
-            <geometry>
-                <box size="0.26 0.15 0.065"/>
-            </geometry>
-        </collision>
-        <xacro:inertial_box mass="0.5" x="0.26" y="0.1" z="0.065">
-            <origin xyz="0.13 0 0.0325" rpy="0 0 0"/>
+            <origin xyz="0.13 0 0.04"/>
+            <geometry>
+                <box size="0.26 0.15 0.08"/>
+            </geometry>
+        </collision>
+        <xacro:inertial_box mass="0.5" x="0.26" y="0.15" z="0.08">
+            <origin xyz="0.13 0 0.04" rpy="0 0 0"/>
         </xacro:inertial_box>
     </link>
@@ -66,14 +66,14 @@
         <visual>
             <geometry>
-                <cylinder radius="0.03" length="0.026"/>
-            </geometry>
-            <material name="blue"/>
-        </visual>
-        <collision>
-            <geometry>
-                <sphere radius="0.03" />
-            </geometry>
-        </collision>
-        <xacro:inertial_cylinder mass="0.1" length="0.026" radius="0.03">
+                <cylinder radius="0.0325" length="0.028"/>
+            </geometry>
+            <material name="blue"/>
+        </visual>
+        <collision>
+            <geometry>
+                <cylinder radius="0.0325" length="0.028"/>
+            </geometry>
+        </collision>
+        <xacro:inertial_cylinder mass="0.1" length="0.028" radius="0.0325">
             <origin xyz="0 0 0" rpy="0 0 0"/>
         </xacro:inertial_cylinder>
@@ -91,14 +91,14 @@
         <visual>
             <geometry>
-                <cylinder radius="0.03" length="0.026"/>
-            </geometry>
-            <material name="blue"/>
-        </visual>
-        <collision>
-            <geometry>
-                <sphere radius="0.03" />
-            </geometry>
-        </collision>
-        <xacro:inertial_cylinder mass="0.1" length="0.026" radius="0.03">
+                <cylinder radius="0.0325" length="0.028"/>
+            </geometry>
+            <material name="blue"/>
+        </visual>
+        <collision>
+            <geometry>
+                <cylinder radius="0.0325" length="0.028" />
+            </geometry>
+        </collision>
+        <xacro:inertial_cylinder mass="0.1" length="0.028" radius="0.0325">
             <origin xyz="0 0 0" rpy="0 0 0"/>
         </xacro:inertial_cylinder>
@@ -106,6 +106,6 @@
     <gazebo reference="left_wheel_front">
         <material>Gazebo/Blue</material>
-        <mu1 value="0.001"/>
-        <mu2 value="0.001"/>
+        <mu1 value="1.0"/>
+        <mu2 value="1.0"/>
     </gazebo>
     <!-- RIGHT WHEEL LINK -->
@@ -119,14 +119,14 @@
         <visual>
             <geometry>
-                <cylinder radius="0.03" length="0.026"/>
-            </geometry>
-            <material name="blue"/>
-        </visual>
-        <collision>
-            <geometry>
-                <sphere radius="0.03" />
-            </geometry>
-        </collision>
-        <xacro:inertial_cylinder mass="0.1" length="0.026" radius="0.03">
+                <cylinder radius="0.0325" length="0.026"/>
+            </geometry>
+            <material name="blue"/>
+        </visual>
+        <collision>
+            <geometry>
+                <cylinder radius="0.0325" length="0.028"/>
+            </geometry>
+        </collision>
+        <xacro:inertial_cylinder mass="0.1" length="0.028" radius="0.0325">
             <origin xyz="0 0 0" rpy="0 0 0"/>
         </xacro:inertial_cylinder>
@@ -144,14 +144,14 @@
         <visual>
             <geometry>
-                <cylinder radius="0.03" length="0.026"/>
-            </geometry>
-            <material name="blue"/>
-        </visual>
-        <collision>
-            <geometry>
-                <sphere radius="0.03" />
-            </geometry>
-        </collision>
-        <xacro:inertial_cylinder mass="0.1" length="0.026" radius="0.03">
+                <cylinder radius="0.0325" length="0.028"/>
+            </geometry>
+            <material name="blue"/>
+        </visual>
+        <collision>
+            <geometry>
+                <cylinder radius="0.0325" length="0.028" />
+            </geometry>
+        </collision>
+        <xacro:inertial_cylinder mass="0.1" length="0.028" radius="0.0325">
             <origin xyz="0 0 0" rpy="0 0 0"/>
         </xacro:inertial_cylinder>
@@ -159,6 +159,6 @@
     <gazebo reference="right_wheel_front">
         <material>Gazebo/Blue</material>
-        <mu1 value="0.001"/>
-        <mu2 value="0.001"/>
+        <mu1 value="1.0"/>
+        <mu2 value="1.0"/>
     </gazebo>
     <!-- Camera Joint -->

File: description/ros2_control.xacro (robot description, xacro)
@@ -1,5 +1,33 @@
 <?xml version="1.0"?>
 <robot xmlns:xacro="http://www.ros.org/wiki/xacro">
-    <ros2_control name="GazeboSystem" type="system">
+    <ros2_control name="RealRobot" type="system">
+        <hardware>
+            <plugin>diffdrive_arduino/DiffDriveArduino</plugin>
+            <param name="left_wheel_name">left_wheel_joint</param>
+            <param name="right_wheel_name">right_wheel_joint</param>
+            <param name="loop_rate">30</param>
+            <param name="device">/dev/ttyACM0</param>
+            <param name="baud_rate">57600</param>
+            <param name="timeout">1000</param>
+            <param name="enc_counts_per_rev">1950</param>
+        </hardware>
+        <joint name="left_wheel_joint">
+            <command_interface name="velocity">
+                <param name="min">-5</param>
+                <param name="max">5</param>
+            </command_interface>
+            <state_interface name="velocity"/>
+            <state_interface name="position"/>
+        </joint>
+        <joint name="right_wheel_joint">
+            <command_interface name="velocity">
+                <param name="min">-5</param>
+                <param name="max">5</param>
+            </command_interface>
+            <state_interface name="velocity"/>
+            <state_interface name="position"/>
+        </joint>
+    </ros2_control>
+    <!-- <ros2_control name="GazeboSystem" type="system">
         <hardware>
             <plugin>gazebo_ros2_control/GazeboSystem</plugin>
@@ -21,5 +49,5 @@
             <state_interface name="position"/>
         </joint>
-    </ros2_control>
+    </ros2_control> -->
     <gazebo>
         <plugin name="gazebo_ros2_control" filename="libgazebo_ros2_control.so">
